File: sismin_baremetal_atmega328p.kicad_pcb (KiCad board)
At the start: 2 copper layers, 24 parts, among them J1 Barrel_Jack_Switch, J2 Conn_01x06_Socket, J3 Conn_01x10_Socket, J4 Conn_01x05_Socket, J5 Conn_01x08_Socket, J6 Conn_02x05_Top_Bottom, SW1 SW_Push, U1 ATmega328-P, U2 LM7805_TO220, Y1 Crystal_Small

Commit message: update
Parts:
- D2: value LED -> LED_POWER
- J1: footprint Connector_BarrelJack:BarrelJack_Wuerth_6941xx301002 -> Connector_BarrelJack:BarrelJack_Horizontal
- moved R1 156.8 mm to (55.6, 22.1)
- moved D2 139.6 mm to (58.8, 50.1)
- moved C4 129.2 mm to (26.0, 70.2)
- moved C5 129.2 mm to (26.0, 73.3)
- moved SW1 122.9 mm to (93.2, 42.5)
- moved D1 117.0 mm to (64.9, 72.0)
- moved Y1 113.1 mm to (27.5, 65.9)
- moved R5 109.3 mm to (55.6, 38.4)
- moved R2 109.3 mm to (55.6, 26.2)
- moved R3 109.3 mm to (55.6, 30.2)
- moved R4 109.3 mm to (55.6, 34.3)
- moved D3 105.4 mm to (70.1, 49.1)
- moved D4 105.4 mm to (70.1, 54.6)
- moved D5 95.7 mm to (58.8, 57.6)
- moved J5 83.9 mm to (152.0, 44.2), turned to 90 degrees
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Other:
- board outline added: 85 x 51 mm

Commit message: update
Parts:
- U2: footprint Package_TO_SOT_THT:TO-220F-3_Horizontal_TabDown -> Package_TO_SOT_THT:TO-220-3_Horizontal_TabDown
- Y1: footprint Crystal:Crystal_HC52-U_Vertical -> Crystal:Crystal_HC49-4H_Vertical
- moved Y1 142.9 mm to (168.5, 89.5), turned to 90 degrees
- moved C1 137.5 mm to (162.3, 91.2), turned to 90 degrees
- moved C3 137.1 mm to (162.3, 84.8), turned to 90 degrees
- moved R4 116.0 mm to (147.2, 97.4), turned to 180 degrees
- moved R2 114.0 mm to (147.2, 102.2), turned to 180 degrees
- moved R3 110.8 mm to (147.2, 92.6), turned to 180 degrees
- moved R10 109.9 mm to (147.2, 82.9), turned to 180 degrees
- moved D5 99.9 mm to (143.5, 110.6)
- moved R1 97.4 mm to (139.6, 87.7)
- moved D4 94.4 mm to (157.7, 89.9), turned to 180 degrees
- moved D3 94.0 mm to (157.7, 83.5), turned to 180 degrees
- moved D2 69.9 mm to (125.8, 70.2)
- moved D1 55.4 mm to (111.8, 101.6)
- moved J2 48.2 mm to (188.0, 111.8)
- moved C4 36.6 mm to (134.7, 110.8)
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- renumbered C5 to C1, C1 to C2, C4 to C3, C2 to C4, R5 to R1, R1 to R10, R4 to R2, R2 to R4
Connections:
- C1 pad 1: Net-(C5-Pad1) -> /XTAL2
- C3 pad 1: Net-(C4-Pad1) -> /XTAL1
- Y1 pad 1: Net-(C5-Pad1) -> /XTAL2
- Y1 pad 2: Net-(C4-Pad1) -> /XTAL1
Other:
- board text added: "A0"
- board text added: "A1"
- board text added: "A2"
- board text added: "A3"
- board text added: "A4"
- board text added: "A5"
- board text added: "AREF"
- board text added: "BOKU MENTATION"
- board text added: "D0"
- board text added: "D1"
- board text added: "D10"
- board text added: "D11"
- board text added: "D12"
- board text added: "D13"
- board text added: "D2"
- board text added: "D3"
- board text added: "D4"
- board text added: "D5"
- board text added: "D6"
- board text added: "D7"
- board text added: "D8"
- board text added: "D9"
- board text added: "GND"
- board text added: "IBRAHIM FAUZI RAHMAN 607022400009 D3TK-48-01"
- board text added: "RESET"
- board text added: "VCC"

Commit message: update 241009
Parts:
- moved R1 12.5 mm to (147.2, 97.6), turned to 180 degrees
- moved R4 12.3 mm to (139.6, 87.8), turned to 0 degrees
- moved D1 8.89 mm to (120.5, 100.0), turned to 180 degrees
- moved D5 1.89 mm to (145.0, 111.8), turned to 90 degrees
- moved J1 1.83 mm to (120.0, 107.5)
- moved SW1 1.40 mm to (113.8, 69.2)
- moved J6 1.20 mm to (115.5, 81.3)
- moved D2 0.80 mm to (125.8, 71.0)
- moved R2 0.26 mm to (147.2, 102.5)
- moved R3 0.13 mm to (147.2, 92.7)
Routing:
- net /D4: track 0.00 -> 25.1 mm
- net /D3: track 0.00 -> 25.1 mm
- net /D2: track 0.00 -> 25.1 mm
- net /D0: track 0.00 -> 25.1 mm
- net /D1: track 0.00 -> 25.1 mm
- net VCC: track 0.00 -> 19.9 mm
- net GND: track 0.00 -> 18.8 mm
- net Net-(D1-K): track 0.00 -> 16.2 mm
- net Net-(D1-A): track 0.00 -> 12.4 mm
- net Net-(D5-A): track 0.00 -> 11.3 mm
- net Net-(U2-VO): track 0.00 -> 11.0 mm
- net /XTAL2: track 0.00 -> 11.0 mm
- net /A4: track 0.00 -> 8.97 mm
- net /A3: track 0.00 -> 8.97 mm
- net /A0: track 0.00 -> 8.97 mm
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
Commit message: update 241009
Parts:
- moved R4 9.06 mm to (147.2, 92.7), turned to 180 degrees
- moved R3 4.90 mm to (147.2, 87.8)
Routing:
- net /D13: track 0.00 -> 81.5 mm
- net VCC: track 19.9 -> 87.4 mm
- net /D12: track 0.00 -> 60.5 mm
- net /RESET: track 6.50 -> 57.4 mm
- net /D11: track 0.00 -> 47.8 mm, vias 0 -> 2
- net Net-(D2-A): track 0.00 -> 20.0 mm
- net Net-(D3-A): track 0.00 -> 14.5 mm
- net Net-(D4-A): track 0.00 -> 9.23 mm
- net /D4: track 25.1 -> 27.2 mm
- net /D0: track 25.1 -> 26.4 mm
- net /D3: track 25.1 -> 25.9 mm

Commit message: update 251013
Routing:
- net /D1: track 25.1 -> 75.9 mm, vias 0 -> 1
- net /D10: track 0.00 -> 41.6 mm, vias 0 -> 1
- net /D5: track 0.00 -> 38.8 mm, vias 0 -> 2
- net /D0: track 26.4 -> 64.4 mm, vias 0 -> 2
- net /D12: track 60.5 -> 98.3 mm, vias 0 -> 4
- net /D11: track 47.8 -> 83.1 mm, vias 2 -> 3
- net /D6: track 0.00 -> 33.7 mm, vias 0 -> 2
- net /D7: track 0.00 -> 33.1 mm
- net /D8: track 0.00 -> 33.0 mm
- net /XTAL1: track 6.26 -> 18.8 mm

Commit message: update 251016
Parts:
- D2: value LED_POWER -> POWER
- D3: value LED_RX -> RX
- D4: value LED_TX -> TX
Connections:
- U1 pad 22: Net-(U1-GND-Pad22) -> GND
- U1 pad 8: Net-(U1-GND-Pad22) -> GND
Routing:
- net /A5: track 9.02 -> 91.5 mm, vias 0 -> 5
- net /RESET: track 57.1 -> 137.4 mm, vias 0 -> 3
- net /A4: track 8.97 -> 87.7 mm, vias 0 -> 5
- net /AREF: track 0.00 -> 63.2 mm, vias 0 -> 2
- net /D9: track 0.00 -> 43.2 mm, vias 0 -> 1
- net Net-(U2-VO): track 11.0 -> 39.4 mm, vias 0 -> 1
- net /D13: track 81.6 -> 105.9 mm, vias 0 -> 3
- net VCC: track 87.4 -> 101.0 mm, vias 0 -> 1
- net /A2: track 8.97 -> 10.1 mm
- net /D12: track 98.3 -> 97.3 mm, vias 4 -> 2
- net /D8: track 33.0 -> 33.7 mm
- net /D7: track 33.1 -> 33.7 mm
- net /A0: track 8.97 -> 9.54 mm
- net /D5: vias 2 -> 1
- net (no net): vias 1 -> 0
- added copper zone on B.Cu, net GND
- added copper zone on F.Cu, net GND
Other:
- board text added: "Check our GitHub: Bokumentation Zidanes-Hub"
- board text removed: "IBRAHIM FAUZI RAHMAN 607022400009 D3TK-48-01"

Commit message: update
Other:
- board text added: "Check our GitHub: - Bokumentation - Zidanes-Hub"
- board text removed: "Check our GitHub: Bokumentation Zidanes-Hub"

Commit message: update 251016
Parts:
- D2: value POWER -> LED_POWER
- D3: value RX -> LED_RX; footprint LED_THT:LED_D3.0mm -> LED_THT:LED_D5.0mm
- D4: value TX -> LED_TX; footprint LED_THT:LED_D3.0mm -> LED_THT:LED_D5.0mm
Changed lines of the file:
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@@
 	(net 34 "/XTAL2")
 	(net 35 "/XTAL1")
-	(footprint "LED_THT:LED_D3.0mm"
+	(footprint "LED_THT:LED_D5.0mm"
 		(layer "F.Cu")
 		(at 157.67 89.94 180)
-		(descr "LED, diameter 3.0mm, 2 pins, generated by kicad-footprint-generator")
+		(descr "LED, diameter 5.0mm, 2 pins, http://cdn-reichelt.de/documents/datenblatt/A500/LL-504BC2E-009.pdf, generated by kicad-footprint-generator")
 		(tags "LED")
 		(property "Reference" "D4"
-			(at -1.69 0 90)
+			(at 1.27 -3.96 180)
 			(layer "F.SilkS")
-			(hide yes)
 			(effects
 				(font
@@
 			)
 		)
-		(property "Value" "TX"
-			(at 4.57 0 180)
-			(layer "F.SilkS")
+		(property "Value" "LED_TX"
+			(at 1.27 3.96 180)
+			(layer "F.Fab")
 			(effects
 				(font
@@
 		)
 		(property "Datasheet" ""
-			(at 0 0 0)
+			(at 0 0 180)
 			(layer "F.Fab")
 			(hide yes)
@@
 		)
 		(property "Description" "Light emitting diode"
-			(at 0 0 0)
+			(at 0 0 180)
 			(layer "F.Fab")
 			(hide yes)
@@
 		(attr through_hole)
 		(fp_line
-			(start -0.29 1.08)
-			(end -0.29 1.236)
-			(stroke
-				(width 0.12)
-				(type solid)
-			)
-			(layer "F.SilkS")
-		)
-		(fp_line
-			(start -0.29 -1.236)
-			(end -0.29 -1.08)
-			(stroke
-				(width 0.12)
-				(type solid)
-			)
-			(layer "F.SilkS")
-		)
-		(fp_arc
-			(start 2.941437 1.08)
-			(mid 1.36566 1.987699)
-			(end -0.29 1.235516)
+			(start -1.29 -1.545)
+			(end -1.29 1.545)
 			(stroke
 				(width 0.12)
@@
 		)
 		(fp_arc
-			(start 2.310961 1.08)
-			(mid 1.27 1.5)
-			(end 0.229039 1.08)
+			(start 4.26 0)
+			(mid 2.071779 2.880495)
+			(end -1.29 1.54483)
 			(stroke
 				(width 0.12)
@@
 		)
 		(fp_arc
-			(start 0.229039 -1.08)
-			(mid 1.27 -1.5)
-			(end 2.310961 -1.08)
+			(start -1.29 -1.54483)
+			(mid 2.071779 -2.880495)
+			(end 4.26 0)
 			(stroke
 				(width 0.12)
@@
 			(layer "F.SilkS")
 		)
-		(fp_arc
-			(start -0.29 -1.235516)
-			(mid 1.36566 -1.987699)
-			(end 2.941437 -1.08)
+		(fp_circle
+			(center 1.27 0)
+			(end 3.77 0)
 			(stroke
 				(width 0.12)
 				(type solid)
 			)
+			(fill no)
 			(layer "F.SilkS")
 		)
 		(fp_line
-			(start 3.69 2.21)
-			(end 3.69 -2.21)
+			(start 4.49 3.21)
+			(end 4.49 -3.21)
 			(stroke
 				(width 0.05)
@@
 		)
 		(fp_line
-			(start 3.69 -2.21)
-			(end -1.15 -2.21)
+			(start 4.49 -3.21)
+			(end -1.94 -3.21)
 			(stroke
 				(width 0.05)
@@
 		)
 		(fp_line
-			(start -1.15 2.21)
-			(end 3.69 2.21)
+			(start -1.94 3.21)
+			(end 4.49 3.21)
 			(stroke
 				(width 0.05)
@@
 		)
 		(fp_line
-			(start -1.15 -2.21)
-			(end -1.15 2.21)
+			(start -1.94 -3.21)
+			(end -1.94 3.21)
 			(stroke
 				(width 0.05)
@@
 		)
 		(fp_line
-			(start -0.23 -1.16619)
-			(end -0.23 1.16619)
+			(start -1.23 -1.469694)
+			(end -1.23 1.469694)
 			(stroke
 				(width 0.1)
@@
 		)
 		(fp_arc
-			(start -0.23 -1.16619)
-			(mid 3.17 0)
-			(end -0.23 1.16619)
+			(start -1.23 -1.469694)
+			(mid 4.17 0)
+			(end -1.23 1.469694)
 			(stroke
 				(width 0.1)
@@
 		(fp_circle
 			(center 1.27 0)
-			(end 2.77 0)
+			(end 3.77 0)
 			(stroke
 				(width 0.1)
@@
 		)
 		(fp_text user "${REFERENCE}"
-			(at 1.27 0 0)
-			(layer "F.SilkS")
+			(at 1.27 0 180)
+			(layer "F.Fab")
 			(effects
 				(font
@@
 		)
 		(embedded_fonts no)
-		(model "${KICAD9_3DMODEL_DIR}/LED_THT.3dshapes/LED_D3.0mm.step"
+		(model "${KICAD9_3DMODEL_DIR}/LED_THT.3dshapes/LED_D5.0mm.step"
 			(offset
 				(xyz 0 0 0)
@@
 			)
 		)
-		(property "Value" "POWER"
+		(property "Value" "LED_POWER"
 			(at 1.27 3.96 0)
 			(layer "F.SilkS")
@@
 		)
 	)
-	(footprint "LED_THT:LED_D3.0mm"
+	(footprint "LED_THT:LED_D5.0mm"
 		(layer "F.Cu")
 		(at 157.67 83.5 180)
-		(descr "LED, diameter 3.0mm, 2 pins, generated by kicad-footprint-generator")
+		(descr "LED, diameter 5.0mm, 2 pins, http://cdn-reichelt.de/documents/datenblatt/A500/LL-504BC2E-009.pdf, generated by kicad-footprint-generator")
 		(tags "LED")
 		(property "Reference" "D3"
-			(at -1.69 0 90)
+			(at 1.27 -3.96 180)
 			(layer "F.SilkS")
-			(hide yes)
 			(effects
 				(font
@@
 			)
 		)
-		(property "Value" "RX"
-			(at 4.57 0 0)
-			(layer "F.SilkS")
+		(property "Value" "LED_RX"
+			(at 1.27 3.96 180)
+			(layer "F.Fab")
 			(effects
 				(font
@@
 		)
 		(property "Datasheet" ""
-			(at 0 0 0)
+			(at 0 0 180)
 			(layer "F.Fab")
 			(hide yes)
@@
 		)
 		(property "Description" "Light emitting diode"
-			(at 0 0 0)
+			(at 0 0 180)
 			(layer "F.Fab")
 			(hide yes)
@@
 		(attr through_hole)
 		(fp_line
-			(start -0.29 1.08)
-			(end -0.29 1.236)
-			(stroke
-				(width 0.12)
-				(type solid)
-			)
-			(layer "F.SilkS")
-		)
-		(fp_line
-			(start -0.29 -1.236)
-			(end -0.29 -1.08)
-			(stroke
-				(width 0.12)
-				(type solid)
-			)
-			(layer "F.SilkS")
-		)
-		(fp_arc
-			(start 2.941437 1.08)
-			(mid 1.36566 1.987699)
-			(end -0.29 1.235516)
+			(start -1.29 -1.545)
+			(end -1.29 1.545)
 			(stroke
 				(width 0.12)
@@
 		)
 		(fp_arc
-			(start 2.310961 1.08)
-			(mid 1.27 1.5)
-			(end 0.229039 1.08)
+			(start 4.26 0)
+			(mid 2.071779 2.880495)
+			(end -1.29 1.54483)
 			(stroke
 				(width 0.12)
@@
 		)
 		(fp_arc
-			(start 0.229039 -1.08)
-			(mid 1.27 -1.5)
-			(end 2.310961 -1.08)
+			(start -1.29 -1.54483)
+			(mid 2.071779 -2.880495)
+			(end 4.26 0)
 			(stroke
 				(width 0.12)
@@
 			(layer "F.SilkS")
 		)
-		(fp_arc
-			(start -0.29 -1.235516)
-			(mid 1.36566 -1.987699)
-			(end 2.941437 -1.08)
+		(fp_circle
+			(center 1.27 0)
+			(end 3.77 0)
 			(stroke
 				(width 0.12)
 				(type solid)
 			)
+			(fill no)
 			(layer "F.SilkS")
 		)
 		(fp_line
-			(start 3.69 2.21)
-			(end 3.69 -2.21)
+			(start 4.49 3.21)
+			(end 4.49 -3.21)
 			(stroke
 				(width 0.05)
@@
 		)
 		(fp_line
-			(start 3.69 -2.21)
-			(end -1.15 -2.21)
+			(start 4.49 -3.21)
+			(end -1.94 -3.21)
 			(stroke
 				(width 0.05)
@@
 		)
 		(fp_line
-			(start -1.15 2.21)
-			(end 3.69 2.21)
+			(start -1.94 3.21)
+			(end 4.49 3.21)
 			(stroke
 				(width 0.05)
@@
 		)
 		(fp_line
-			(start -1.15 -2.21)
-			(end -1.15 2.21)
+			(start -1.94 -3.21)
+			(end -1.94 3.21)
 			(stroke
 				(width 0.05)
@@
 		)
 		(fp_line
-			(start -0.23 -1.16619)
-			(end -0.23 1.16619)
+			(start -1.23 -1.469694)
+			(end -1.23 1.469694)
 			(stroke
 				(width 0.1)
@@
 		)
 		(fp_arc
-			(start -0.23 -1.16619)
-			(mid 3.17 0)
-			(end -0.23 1.16619)
+			(start -1.23 -1.469694)
+			(mid 4.17 0)
+			(end -1.23 1.469694)
 			(stroke
 				(width 0.1)
@@
 		(fp_circle
 			(center 1.27 0)
-			(end 2.77 0)
+			(end 3.77 0)
 			(stroke
 				(width 0.1)
@@
 		)
 		(fp_text user "${REFERENCE}"
-			(at 1.27 0 0)
-			(layer "F.SilkS")
+			(at 1.27 0 180)
+			(layer "F.Fab")
 			(effects
 				(font
@@
 		)
 		(embedded_fonts no)
-		(model "${KICAD9_3DMODEL_DIR}/LED_THT.3dshapes/LED_D3.0mm.step"
+		(model "${KICAD9_3DMODEL_DIR}/LED_THT.3dshapes/LED_D5.0mm.step"
 			(offset
 				(xyz 0 0 0)
