File: sismin_baremetal_atmega328p.kicad_sch (KiCad schematic)
At the start: 24 parts, among them J1 Barrel_Jack_Switch, J2 Conn_01x06_Socket, J3 Conn_01x10_Socket, J4 Conn_01x05_Socket, J5 Conn_01x08_Socket, J6 Conn_02x05_Top_Bottom, SW1 SW_Push, U1 ATmega328-P, U2 LM7805_TO220, Y1 Crystal_Small

Commit message: update
Parts:
- D2: value LED -> LED_POWER
- J1: footprint Connector_BarrelJack:BarrelJack_Wuerth_6941xx301002 -> Connector_BarrelJack:BarrelJack_Horizontal
Other:
- moved on the sheet: C1, C2, C4, C5, D1, D2, D3, D4, D5, J1, J2, J3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

Commit message: update
Parts:
- U2: footprint Package_TO_SOT_THT:TO-220F-3_Horizontal_TabDown -> Package_TO_SOT_THT:TO-220-3_Horizontal_TabDown
- Y1: footprint Crystal:Crystal_HC52-U_Vertical -> Crystal:Crystal_HC49-4H_Vertical
- renumbered C5 to C1, C1 to C2, C4 to C3, C2 to C4, R5 to R1, R1 to R10, R4 to R2, R2 to R4
Connections:
- net XTAL1: now also C3.1, Y1.2
- net XTAL2: now also C1.1, Y1.1
Changed lines of the file:
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@@
 	)
 	(junction
+		(at 36.83 41.91)
+		(diameter 0)
+		(color 0 0 0 0)
+	)
+	(junction
 		(at 245.11 27.94)
 		(diameter 0)
@@
 	)
 	(junction
+		(at 36.83 29.21)
+		(diameter 0)
+		(color 0 0 0 0)
+	)
+	(junction
 		(at 19.05 41.91)
 		(diameter 0)
@@
 	)
 	(bus_entry
+		(at 53.34 24.13)
+		(size -2.54 2.54)
+		(stroke
+			(width 0)
+			(type default)
+		)
+	)
+	(bus_entry
 		(at 53.34 41.91)
 		(size 2.54 2.54)
@@
 	)
 	(bus_entry
+		(at 53.34 27.94)
+		(size -2.54 2.54)
+		(stroke
+			(width 0)
+			(type default)
+		)
+	)
+	(bus_entry
 		(at 53.34 34.29)
 		(size 2.54 2.54)
@@
 		)
 	)
+	(wire
+		(pts
+			(xy 50.8 30.48) (xy 50.8 41.91)
+		)
+		(stroke
+			(width 0)
+			(type default)
+		)
+	)
 	(bus
 		(pts
@@
 		)
 	)
+	(bus
+		(pts
+			(xy 53.34 27.94) (xy 53.34 24.13)
+		)
+		(stroke
+			(width 0)
+			(type default)
+		)
+	)
 	(wire
 		(pts
@@
 	(bus
 		(pts
+			(xy 53.34 24.13) (xy 53.34 21.59)
+		)
+		(stroke
+			(width 0)
+			(type default)
+		)
+	)
+	(bus
+		(pts
 			(xy 77.47 107.95) (xy 67.31 107.95)
 		)
@@
 	(wire
 		(pts
+			(xy 50.8 26.67) (xy 36.83 26.67)
+		)
+		(stroke
+			(width 0)
+			(type default)
+		)
+	)
+	(wire
+		(pts
 			(xy 36.83 78.74) (xy 36.83 83.82)
 		)
@@
 	(bus
 		(pts
-			(xy 53.34 31.75) (xy 53.34 21.59)
+			(xy 53.34 31.75) (xy 53.34 27.94)
 		)
 		(stroke
@@
 		)
 	)
+	(wire
+		(pts
+			(xy 36.83 26.67) (xy 36.83 29.21)
+		)
+		(stroke
+			(width 0)
+			(type default)
+		)
+	)
 	(bus
 		(pts
@@
 	(wire
 		(pts
+			(xy 50.8 41.91) (xy 36.83 41.91)
+		)
+		(stroke
+			(width 0)
+			(type default)
+		)
+	)
+	(wire
+		(pts
 			(xy 50.8 97.79) (xy 34.29 97.79)
 		)
@@
 		)
 	)
+	(label "XTAL1"
+		(at 36.83 41.91 0)
+		(effects
+			(font
+				(size 1.27 1.27)
+			)
+			(justify left bottom)
+		)
+	)
 	(label "D1"
 		(at 64.77 49.53 0)
@@
 		)
 	)
+	(label "XTAL2"
+		(at 36.83 26.67 0)
+		(effects
+			(font
+				(size 1.27 1.27)
+			)
+			(justify left bottom)
+		)
+	)
 	(label "D5"
 		(at 133.35 96.52 0)
@@
 		(dnp no)
 		(fields_autoplaced yes)
-		(property "Reference" "C5"
+		(property "Reference" "C1"
 			(at 26.67 21.59 90)
 			(effects
@@
 			(project "sismin_baremetal_atmega328p"
 				(path "/6dafda5e-5668-4e33-8bc1-7d1abbf48d06"
-					(reference "C5")
+					(reference "C1")
 					(unit 1)
 				)
@@
 		(dnp no)
 		(fields_autoplaced yes)
-		(property "Reference" "R4"
+		(property "Reference" "R2"
 			(at 30.48 92.7099 0)
 			(effects
@@
 			(project "sismin_baremetal_atmega328p"
 				(path "/6dafda5e-5668-4e33-8bc1-7d1abbf48d06"
-					(reference "R4")
+					(reference "R2")
 					(unit 1)
 				)
@@
 		(dnp no)
 		(fields_autoplaced yes)
-		(property "Reference" "R5"
+		(property "Reference" "R1"
 			(at 39.37 59.6899 0)
 			(effects
@@
 			(project "sismin_baremetal_atmega328p"
 				(path "/6dafda5e-5668-4e33-8bc1-7d1abbf48d06"
-					(reference "R5")
+					(reference "R1")
 					(unit 1)
 				)
@@
 		(on_board yes)
 		(dnp no)
-		(property "Reference" "C2"
+		(property "Reference" "C4"
 			(at 248.92 39.7509 0)
 			(effects
@@
 			(project ""
 				(path "/6dafda5e-5668-4e33-8bc1-7d1abbf48d06"
-					(reference "C2")
+					(reference "C4")
 					(unit 1)
 				)
@@
 		(dnp no)
 		(fields_autoplaced yes)
-		(property "Reference" "C4"
+		(property "Reference" "C3"
 			(at 26.67 34.29 90)
 			(effects
@@
 			(project ""
 				(path "/6dafda5e-5668-4e33-8bc1-7d1abbf48d06"
-					(reference "C4")
+					(reference "C3")
 					(unit 1)
 				)
@@
 		(dnp no)
 		(fields_autoplaced yes)
-		(property "Reference" "R2"
+		(property "Reference" "R4"
 			(at 64.77 134.6199 0)
 			(effects
@@
 			(project "sismin_baremetal_atmega328p"
 				(path "/6dafda5e-5668-4e33-8bc1-7d1abbf48d06"
-					(reference "R2")
+					(reference "R4")
 					(unit 1)
 				)
@@
 			)
 		)
-		(property "Footprint" "Crystal:Crystal_HC52-U_Vertical"
+		(property "Footprint" "Crystal:Crystal_HC49-4H_Vertical"
 			(at 36.83 35.56 0)
 			(effects
@@
 		(dnp no)
 		(fields_autoplaced yes)
-		(property "Reference" "C1"
+		(property "Reference" "C2"
 			(at 218.44 39.7509 0)
 			(effects
@@
 			(project ""
 				(path "/6dafda5e-5668-4e33-8bc1-7d1abbf48d06"
-					(reference "C1")
+					(reference "C2")
 					(unit 1)
 				)
@@
 		(dnp no)
 		(fields_autoplaced yes)
-		(property "Reference" "R1"
+		(property "Reference" "R10"
 			(at 270.51 30.4799 0)
 			(effects
@@
 			(project ""
 				(path "/6dafda5e-5668-4e33-8bc1-7d1abbf48d06"
-					(reference "R1")
+					(reference "R10")
 					(unit 1)
 				)
@@
 			)
 		)
-		(property "Footprint" "Package_TO_SOT_THT:TO-220F-3_Horizontal_TabDown"
+		(property "Footprint" "Package_TO_SOT_THT:TO-220-3_Horizontal_TabDown"
 			(at 229.87 22.225 0)
 			(effects

Commit message: update 251016
Connections:
- net GND: now also U1.22 (GND), U1.8 (GND)
Changed lines of the file:
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@@
+	)
+	(bus_entry
+		(at 121.92 24.13)
+		(size -2.54 2.54)
+		(stroke
+			(width 0)
+			(type default)
+		)
 	)
 	(bus_entry
@@
 	(wire
 		(pts
+			(xy 87.63 26.67) (xy 119.38 26.67)
+		)
+		(stroke
+			(width 0)
+			(type default)
+		)
+	)
+	(wire
+		(pts
 			(xy 43.18 69.85) (xy 43.18 67.31)
 		)
@@
 	(bus
 		(pts
+			(xy 121.92 24.13) (xy 121.92 27.94)
+		)
+		(stroke
+			(width 0)
+			(type default)
+		)
+	)
+	(bus
+		(pts
 			(xy 55.88 107.95) (xy 53.34 107.95)
 		)
@@
 	(bus
 		(pts
-			(xy 121.92 21.59) (xy 121.92 27.94)
+			(xy 121.92 21.59) (xy 121.92 24.13)
 		)
 		(stroke
@@
 		(effects
 			(font
+				(size 1.27 1.27)
+			)
+			(justify left bottom)
+		)
+	)
+	(label "GND"
+		(at 87.63 26.67 0)
+		(effects
+			(font

Commit message: update 251016
Parts:
- D3, D4: footprint LED_THT:LED_D3.0mm -> LED_THT:LED_D5.0mm
Changed lines of the file:
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@@
 			)
 		)
-		(property "Footprint" "LED_THT:LED_D3.0mm"
+		(property "Footprint" "LED_THT:LED_D5.0mm"
 			(at 62.23 124.46 0)
 			(effects
@@
 			)
 		)
-		(property "Footprint" "LED_THT:LED_D3.0mm"
+		(property "Footprint" "LED_THT:LED_D5.0mm"
 			(at 48.26 124.46 0)
 			(effects
